Commit message: use 2025-10v for amr_sweeper_description

File: src/amr_sweeper_description/urdf/amr_sweeper.urdf.xacro (robot description, xacro)
@@ -1,8 +1,8 @@
 <?xml version="1.0"?>
-<robot xmlns:xacro="http://www.ros.org/wiki/xacro"  name="AMRSweeper">
+<robot xmlns:xacro="http://www.ros.org/wiki/xacro"  name="amr_sweeper">
     <xacro:include filename="materials.xacro" />
     <xacro:include filename="robot_core.xacro" />
-    <xacro:include filename="GNSS_sensor.xacro" />
-    <xacro:include filename="IMU_sensor.xacro" />
+    <xacro:include filename="gnss_sensor.xacro" />
+    <xacro:include filename="imu_sensor.xacro" />
     <xacro:include filename="depth_camera.xacro" />
     <xacro:arg name="use_ros2_control" default="true"/>

File: src/amr_sweeper_description/urdf/gazebo_control.xacro (robot description, xacro)
@@ -4,16 +4,16 @@
         <plugin
             filename="gz-sim-diff-drive-system"
-            name="gz::sim::systems::DiffDrive" >
-            <!-- Wheel Information -->
-            <left_joint>LeftWheel_joint</left_joint>
-            <right_joint>RightWheel_joint</right_joint>
+            name="gz::sim::systems::DiffDrive">
+            <!-- wheel information -->
+            <left_joint>left_wheel_joint</left_joint>
+            <right_joint>right_wheel_joint</right_joint>
             <wheel_separation>0.488</wheel_separation>
             <wheel_radius>0.130</wheel_radius>
-            <!-- Limits -->
+            <!-- limits -->
             <max_wheel_torque>200</max_wheel_torque>
             <max_linear_acceleration>0.33</max_linear_acceleration>
-            <!-- Input -->
+            <!-- input -->
             <topic>cmd_vel</topic>
-            <!-- Output -->
+            <!-- output -->
             <frame_id>odom</frame_id>
             <child_frame_id>base_link</child_frame_id>
@@ -25,7 +25,7 @@
             filename="gz-sim-joint-state-publisher-system"
             name="gz::sim::systems::JointStatePublisher">
-                <topic>joint_states</topic>
-                <joint_name>LeftWheel_joint</joint_name>
-                <joint_name>RightWheel_joint</joint_name>
+            <topic>joint_states</topic>
+            <joint_name>left_wheel_joint</joint_name>
+            <joint_name>right_wheel_joint</joint_name>
         </plugin>
     </gazebo>

File: src/amr_sweeper_description/urdf/robot_core.xacro (robot description, xacro)
@@ -1,51 +1,49 @@
 <?xml version="1.0"?>
 <robot xmlns:xacro="http://www.ros.org/wiki/xacro">
-    <link name="base_link">
-    </link>
+    <link name="base_link"/>
     <joint name="base_footprint_joint" type="fixed">
-        <parent link="base_link" />
-        <child  link="base_footprint" />
+        <parent link="base_link"/>
+        <child link="base_footprint"/>
         <origin xyz="0 0 -0.13" rpy="0 0 0"/>
     </joint>
-    <link name="base_footprint">
-    </link>
-    <joint name="Chassis_joint" type="fixed">
-        <parent link="base_link" />
-        <child  link="Chassis_link" />
+    <link name="base_footprint"/>
+    <joint name="chassis_joint" type="fixed">
+        <parent link="base_link"/>
+        <child link="chassis_link"/>
         <origin xyz="0 0 0" rpy="0 0 0"/>
     </joint>
-    <link name="Chassis_link">
+    <link name="chassis_link">
         <visual>
             <origin xyz="0 0 0" rpy="0 0 0"/>
             <geometry>
-                <mesh   filename="package://AMR-Sweeper_description/meshes/Chassis/Chassis.stl" />
+                <mesh filename="package://amr_sweeper_description/meshes/chassis/v2025_09/chassis_assembly.stl"/>
             </geometry>
             <material name="grey"/>
         </visual>
-<!--
+        <!--
         <collision>
             <origin xyz="0 0 0" rpy="0 0 0"/>
             <geometry>
-                <mesh   filename="package://AMR-Sweeper_description/meshes/Chassis/Chassis.stl" />
+                <mesh filename="package://amr_sweeper_description/meshes/chassis/v2025_09/chassis_assembly.stl"/>
             </geometry>
         </collision>
--->
+        -->
         <inertial>
             <origin xyz="0.054 0 0.110" rpy="0 0 0"/>
-            <mass value="15.4" />
-            <inertia ixx="0.2" ixy="0.002" ixz="-0.010" iyy="0.376" iyz="0.000" izz="0.508" />
+            <mass value="15.4"/>
+            <inertia ixx="0.2" ixy="0.002" ixz="-0.010" iyy="0.376" iyz="0.000" izz="0.508"/>
         </inertial>
     </link>
-    <joint name="LeftWheel_joint" type="continuous">
-        <parent link="base_link" />
-        <child  link="LeftWheel_link" />
-        <origin xyz="0 0.244 0" rpy="-${pi/2} 0 0" />
-        <axis   xyz="0 0 1" />
+    <joint name="left_wheel_joint" type="continuous">
+        <parent link="base_link"/>
+        <child link="left_wheel_link"/>
+        <origin xyz="0 0.244 0" rpy="-${pi/2} 0 0"/>
+        <axis xyz="0 0 1"/>
     </joint>
-    <link name="LeftWheel_link">
+    <link name="left_wheel_link">
         <visual>
             <origin xyz="0 0 0" rpy="${pi/2} 0 0"/>
             <geometry>
-                <mesh   filename="package://AMR-Sweeper_description/meshes/WheelAssembly/WheelAssembly.stl" />
+                <mesh filename="package://amr_sweeper_description/meshes/wheel_assembly/v2025_09/wheel_assembly.stl"/>
             </geometry>
             <material name="yellow"/>
@@ -54,24 +52,24 @@
             <origin xyz="0 0 0" rpy="${pi/2} 0 0"/>
             <geometry>
-                <mesh   filename="package://AMR-Sweeper_description/meshes/WheelAssembly/WheelAssembly.stl" />
+                <mesh filename="package://amr_sweeper_description/meshes/wheel_assembly/v2025_09/wheel_assembly.stl"/>
             </geometry>
         </collision>
         <inertial>
             <origin xyz="0 0 0" rpy="0 0 0"/>
-            <mass value="1.5" />
-            <inertia ixx="0.01" ixy="0" ixz="0" iyy="0.02" iyz="0" izz="0.01" />
+            <mass value="1.5"/>
+            <inertia ixx="0.01" ixy="0" ixz="0" iyy="0.02" iyz="0" izz="0.01"/>
         </inertial>
     </link>
-    <joint name="RightWheel_joint" type="continuous">
-        <parent link="base_link" />
-        <child  link="RightWheel_link" />
-        <origin xyz="0 -0.244 0" rpy="${pi/2} 0 0" />
-        <axis   xyz="0 0 -1" />
+    <joint name="right_wheel_joint" type="continuous">
+        <parent link="base_link"/>
+        <child link="right_wheel_link"/>
+        <origin xyz="0 -0.244 0" rpy="${pi/2} 0 0"/>
+        <axis xyz="0 0 -1"/>
     </joint>
-    <link name="RightWheel_link">
+    <link name="right_wheel_link">
         <visual>
             <origin xyz="0 0 0" rpy="${pi/2} 0 0"/>
             <geometry>
-                <mesh   filename="package://AMR-Sweeper_description/meshes/WheelAssembly/WheelAssembly.stl" />
+                <mesh filename="package://amr_sweeper_description/meshes/wheel_assembly/v2025_09/wheel_assembly.stl"/>
             </geometry>
             <material name="yellow"/>
@@ -80,25 +78,25 @@
             <origin xyz="0 0 0" rpy="${pi/2} 0 0"/>
             <geometry>
-                <mesh   filename="package://AMR-Sweeper_description/meshes/WheelAssembly/WheelAssembly.stl" />
+                <mesh filename="package://amr_sweeper_description/meshes/wheel_assembly/v2025_09/wheel_assembly.stl"/>
             </geometry>
         </collision>
         <inertial>
             <origin xyz="0 0 0" rpy="0 0 0"/>
-            <mass value="1.5" />
-            <inertia ixx="0.01" ixy="0" ixz="0" iyy="0.02" iyz="0" izz="0.01" />
+            <mass value="1.5"/>
+            <inertia ixx="0.01" ixy="0" ixz="0" iyy="0.02" iyz="0" izz="0.01"/>
         </inertial>
     </link>
-    <joint name="Tool_joint" type="fixed">
-        <origin xyz="0.33 0 0.075" rpy="0 0 0" />
-        <parent link="base_link" />
-        <child  link="Tool_link" />
-        <axis   xyz="1 0 0" />
-        <!--<limit  lower="-${pi/18}" upper="${pi/18}" velocity="100" effort="100"/>  -->
+    <joint name="tool_joint" type="fixed">
+        <origin xyz="0.33 0 0.075" rpy="0 0 0"/>
+        <parent link="base_link"/>
+        <child link="tool_link"/>
+        <axis xyz="1 0 0"/>
+        <!--<limit lower="-${pi/18}" upper="${pi/18}" velocity="100" effort="100"/>-->
     </joint>
-    <link name="Tool_link">
+    <link name="tool_link">
         <visual>
             <origin xyz="0 0 0" rpy="0 0 0"/>
             <geometry>
-                <mesh   filename="package://AMR-Sweeper_description/meshes/Tool/Tool.stl" />
+                <mesh filename="package://amr_sweeper_description/meshes/tool/v2025_09/tool_mount.stl"/>
             </geometry>
             <material name="black"/>
@@ -106,18 +104,18 @@
         <inertial>
             <origin xyz="0 0 0" rpy="0 0 0"/>
-            <mass value="2.5" />
-            <inertia ixx="0.01" ixy="0" ixz="0" iyy="0.02" iyz="0" izz="0.01" />
+            <mass value="2.5"/>
+            <inertia ixx="0.01" ixy="0" ixz="0" iyy="0.02" iyz="0" izz="0.01"/>
         </inertial>
     </link>
-    <joint name="LeftBrush_joint" type="fixed">
-        <origin xyz="0 -0.155 -0.073" rpy="0 0 0" />
-        <parent link="Tool_link" />
-        <child  link="LeftBrush_link" />
+    <joint name="left_brush_joint" type="fixed">
+        <origin xyz="0 -0.155 -0.073" rpy="0 0 0"/>
+        <parent link="tool_link"/>
+        <child link="left_brush_link"/>
     </joint>
-    <link name="LeftBrush_link">
+    <link name="left_brush_link">
         <visual>
             <origin xyz="0 0 0" rpy="0 0 0"/>
             <geometry>
-                <mesh   filename="package://AMR-Sweeper_description/meshes/Tool/Brush.stl" />
+                <mesh filename="package://amr_sweeper_description/meshes/tool/v2025_09/nylon_brush.stl"/>
             </geometry>
             <material name="red"/>
@@ -126,23 +124,23 @@
             <origin xyz="0 0 0" rpy="0 0 0"/>
             <geometry>
-                <mesh   filename="package://AMR-Sweeper_description/meshes/Tool/Brush.stl" />
+                <mesh filename="package://amr_sweeper_description/meshes/tool/v2025_09/nylon_brush.stl"/>
             </geometry>
         </collision>
         <inertial>
             <origin xyz="0 0 0" rpy="0 0 0"/>
-            <mass value="1.5" />
-            <inertia ixx="0.01" ixy="0" ixz="0" iyy="0.02" iyz="0" izz="0.01" />
+            <mass value="1.5"/>
+            <inertia ixx="0.01" ixy="0" ixz="0" iyy="0.02" iyz="0" izz="0.01"/>
         </inertial>
     </link>
-    <joint name="RightBrush_joint" type="fixed">
-        <origin xyz="0 0.155 -0.073" rpy="0 0 0" />
-        <parent link="Tool_link" />
-        <child  link="RightBrush_link" />
+    <joint name="right_brush_joint" type="fixed">
+        <origin xyz="0 0.155 -0.073" rpy="0 0 0"/>
+        <parent link="tool_link"/>
+        <child link="right_brush_link"/>
     </joint>
-    <link name="RightBrush_link">
+    <link name="right_brush_link">
         <visual>
             <origin xyz="0 0 0" rpy="0 0 0"/>
             <geometry>
-                <mesh   filename="package://AMR-Sweeper_description/meshes/Tool/Brush.stl" />
+                <mesh filename="package://amr_sweeper_description/meshes/tool/v2025_09/nylon_brush.stl"/>
             </geometry>
             <material name="red"/>
@@ -151,11 +149,11 @@
             <origin xyz="0 0 0" rpy="0 0 0"/>
             <geometry>
-                <mesh   filename="package://AMR-Sweeper_description/meshes/Tool/Brush.stl" />
+                <mesh filename="package://amr_sweeper_description/meshes/tool/v2025_09/nylon_brush.stl"/>
             </geometry>
         </collision>
         <inertial>
             <origin xyz="0 0 0" rpy="0 0 0"/>
-            <mass value="1.5" />
-            <inertia ixx="0.01" ixy="0" ixz="0" iyy="0.02" iyz="0" izz="0.01" />
+            <mass value="1.5"/>
+            <inertia ixx="0.01" ixy="0" ixz="0" iyy="0.02" iyz="0" izz="0.01"/>
         </inertial>
     </link>

File: src/amr_sweeper_description/urdf/ros2_control.xacro (robot description, xacro)
@@ -1,9 +1,9 @@
 <?xml version="1.0"?>
 <robot xmlns:xacro="http://www.ros.org/wiki/xacro">
-    <ros2_control name="RealRobot" type="system">
+    <ros2_control name="real_robot" type="system">
         <hardware>
             <plugin>diffdrive_arduino/DiffDriveArduino</plugin>
-            <param name="left_wheel_name">LeftWheel_joint</param>
-            <param name="right_wheel_name">RightWheel_joint</param>
+            <param name="left_wheel_name">left_wheel_joint</param>
+            <param name="right_wheel_name">right_wheel_joint</param>
             <param name="loop_rate">30</param>
             <param name="device">/dev/ttyUSB0</param>
@@ -12,5 +12,5 @@
             <param name="enc_counts_per_rev">3436</param>
         </hardware>
-        <joint name="LeftWheel_joint">
+        <joint name="left_wheel_joint">
             <command_interface name="velocity">
                 <param name="min">-10</param>
@@ -20,5 +20,5 @@
             <state_interface name="position"/>
         </joint>
-        <joint name="RightWheel_joint">
+        <joint name="right_wheel_joint">
             <command_interface name="velocity">
                 <param name="min">-10</param>
